Commit message: offline slam working

File: urdf/shark_v1.xacro (robot description, xacro)
@@ -1,13 +1,15 @@
 <?xml version="1.0"?>
-<robot xmlns:xacro="http://www.ros.org/wiki/xacro" name="robaka_v2">
-  <xacro:property name="base_width" value="0.3"/>
-  <xacro:property name="base_len" value="0.4"/>
-  <xacro:property name="base_height" value="0.12"/>
-  <xacro:property name="wheel_radius" value="0.085"/>
-  <xacro:property name="base_wheel_gap" value="0.02"/>
-  <xacro:property name="wheel_separation" value="0.31"/>
-  <xacro:property name="wheel_joint_offset" value="-0.107"/>
-  <xacro:property name="caster_wheel_radius" value="0.0375"/>
-  <xacro:property name="caster_wheel_joint_offset" value="0.12"/>
+<robot xmlns:xacro="http://www.ros.org/wiki/xacro" name="shark-v1">
+  <xacro:include filename="$(find doris_sensors_description)/urdf/hokuyo.urdf.xacro" />
+  <xacro:property name="base_width" value="0.531"/>
+  <xacro:property name="base_len" value="0.3785"/>
+  <xacro:property name="base_height" value="0.2895"/>
+  <xacro:property name="wheel_radius" value="0.1"/>
+  <xacro:property name="base_wheel_gap" value="-0.09"/>
+  <xacro:property name="wheel_separation" value="0.35"/>
+  <xacro:property name="wheel_joint_offset" value="-0.005"/>
+  <xacro:property name="caster_height" value="0.060575"/>
+  <!-- <xacro:property name="caster_wheel_radius" value="0.0375"/>
+  <xacro:property name="caster_wheel_joint_offset" value="0.12"/> -->
   <xacro:include filename="$(find shark-mb-ros)/urdf/shark_v1_gazebo_plugins.xacro"/>
   <material name="blue">
@@ -37,5 +39,4 @@
     </inertial>
   </xacro:macro>
-  <link name="dummy"/>
   <link name="base_footprint">
     <xacro:box_inertia m="8" w="0.001" h="0.001" d="0.001"/>
@@ -48,8 +49,4 @@
     </visual>
   </link>
-  <joint name="dummy_joint" type="fixed">
-     <parent link="dummy"/>
-     <child link="base_footprint"/>
-     </joint>
   <link name="base_link">
     <xacro:box_inertia m="1" w="${base_len}" h="${base_width}" d="0.01"/>
@@ -67,5 +64,5 @@
   </link>
   <joint name="base_link_joint" type="fixed">
-    <origin xyz="0 0 ${wheel_radius + 0.005}" rpy="0 0 0" />
+    <origin xyz="0 0 ${base_height/2 + caster_height}" rpy="0 0 0" />
     <parent link="base_footprint"/>
     <child link="base_link" />
@@ -83,5 +80,5 @@
         <origin xyz="0 0 0" rpy="${pi/2} 0 0"/>
         <geometry>
-          <cylinder radius="${wheel_radius}" length="0.02"/>
+          <cylinder radius="${wheel_radius}" length="0.05"/>
         </geometry>
       </visual>
@@ -89,8 +86,8 @@
         <origin xyz="0 0 0" rpy="${pi/2} 0 0"/>
         <geometry>
-          <cylinder radius="${wheel_radius}" length="0.02"/>
+          <cylinder radius="${wheel_radius}" length="0.05"/>
         </geometry>
       </collision>
-      <xacro:cylinder_inertia m="10" r="${wheel_radius}" h="0.02"/>
+      <xacro:cylinder_inertia m="10" r="${wheel_radius}" h="0.05"/>
     </link>
     <joint name="${prefix}_wheel" type="continuous">
@@ -98,5 +95,5 @@
       <parent link="base_link"/>
       <child link="${prefix}_wheel"/>
-      <origin xyz="${wheel_joint_offset} ${((base_width/2)+base_wheel_gap)*reflect} -0.06" rpy="0 0 0"/>
+      <origin xyz="${wheel_joint_offset} ${((base_width/2)+base_wheel_gap)*reflect} ${(wheel_radius - caster_height) - base_height/2}" rpy="0 0 0"/>
     </joint>
   </xacro:macro>
@@ -109,5 +106,5 @@
     </inertial>
   </xacro:macro>
-   <link name="caster_wheel">
+   <!-- <link name="caster_wheel">
      <visual>
        <material name="darkgray"/>
@@ -130,31 +127,5 @@
     <child link="caster_wheel"/>
     <origin xyz="${caster_wheel_joint_offset} 0 -${0.06+caster_wheel_radius}" rpy="0 0 0"/>
-  </joint>
-  <joint name="imu_joint" type="fixed">
-    <parent link="base_link" />
-    <child link="imu" />
-    <origin xyz="0.16 -0.065 0.035" rpy="0 0 0" />
-  </joint>
-  <link name="imu" />
-  <joint name="lidar_joint" type="fixed">
-    <parent link="base_link" />
-    <child link="lidar" />
-    <origin xyz="0.0 0.0 0.12" rpy="0 0 3.14159" />
-  </joint>
-  <link name="lidar">
-    <visual>
-      <material name="blue" />
-      <origin xyz="0 0 0" rpy="0 0 0"/>
-      <geometry>
-        <cylinder radius="0.032" length="0.02"/>
-      </geometry>
-    </visual>
-  </link>
-  <joint name="camera_joint" type="fixed">
-    <origin xyz="0.185 0 0.07" rpy="0 0 3.14159" />
-    <parent link="base_link" />
-    <child link="camera_link" />
-  </joint>
-  <link name="camera_link" type="fixed">
-  </link>
+  </joint> -->
+  <xacro:sensor_hokuyo parent="base_link" xyz="${base_len/2 + 0.025 + 0.0159} 0 ${0.02 - base_height/2}" rpy="0 0 0" />
 </robot>

Commit message: adjusting URDF

File: urdf/shark_v1.xacro (robot description, xacro)
@@ -2,12 +2,12 @@
 <robot xmlns:xacro="http://www.ros.org/wiki/xacro" name="shark-v1">
   <xacro:include filename="$(find doris_sensors_description)/urdf/hokuyo.urdf.xacro" />
-  <xacro:property name="base_width" value="0.531"/>
-  <xacro:property name="base_len" value="0.3785"/>
-  <xacro:property name="base_height" value="0.2895"/>
+  <xacro:property name="base_width" value="0.335"/>
+  <xacro:property name="base_len" value="0.5"/>
+  <xacro:property name="base_height" value="0.3"/>
   <xacro:property name="wheel_radius" value="0.1"/>
-  <xacro:property name="base_wheel_gap" value="-0.09"/>
-  <xacro:property name="wheel_separation" value="0.35"/>
-  <xacro:property name="wheel_joint_offset" value="-0.005"/>
-  <xacro:property name="caster_height" value="0.060575"/>
+  <xacro:property name="base_wheel_gap" value="0.005"/>
+  <xacro:property name="wheel_separation" value="0.36"/>
+  <xacro:property name="wheel_joint_offset" value="0.005"/>
+  <xacro:property name="caster_height" value="0.07"/>
   <!-- <xacro:property name="caster_wheel_radius" value="0.0375"/>
   <xacro:property name="caster_wheel_joint_offset" value="0.12"/> -->

Commit message: fixing URDF

File: urdf/shark_v1.xacro (robot description, xacro)
@@ -1,13 +1,13 @@
 <?xml version="1.0"?>
 <robot xmlns:xacro="http://www.ros.org/wiki/xacro" name="shark-v1">
-  <xacro:include filename="$(find doris_sensors_description)/urdf/hokuyo.urdf.xacro" />
-  <xacro:property name="base_width" value="0.531"/>
-  <xacro:property name="base_len" value="0.3785"/>
-  <xacro:property name="base_height" value="0.2895"/>
+  <xacro:include filename="$(find doris_sensors_description)/urdf/hokuyo.urdf.xacro"/>
+  <xacro:property name="base_width" value="0.335"/>
+  <xacro:property name="base_len" value="0.5"/>
+  <xacro:property name="base_height" value="0.3"/>
   <xacro:property name="wheel_radius" value="0.1"/>
-  <xacro:property name="base_wheel_gap" value="-0.09"/>
-  <xacro:property name="wheel_separation" value="0.35"/>
-  <xacro:property name="wheel_joint_offset" value="-0.005"/>
-  <xacro:property name="caster_height" value="0.060575"/>
+  <xacro:property name="base_wheel_gap" value="0.005"/>
+  <xacro:property name="wheel_separation" value="0.36"/>
+  <xacro:property name="wheel_joint_offset" value="0.0"/>
+  <xacro:property name="caster_height" value="0.07"/>
   <!-- <xacro:property name="caster_wheel_radius" value="0.0375"/>
   <xacro:property name="caster_wheel_joint_offset" value="0.12"/> -->
@@ -40,5 +40,5 @@
   </xacro:macro>
   <link name="base_footprint">
-    <!-- <xacro:box_inertia m="8" w="0.001" h="0.001" d="0.001"/> -->
+    <xacro:box_inertia m="8" w="0.001" h="0.001" d="0.001"/>
     <visual>
       <origin xyz="0 0 0" rpy="0 0 0" />
@@ -128,4 +128,5 @@
     <origin xyz="${caster_wheel_joint_offset} 0 -${0.06+caster_wheel_radius}" rpy="0 0 0"/>
   </joint> -->
-  <xacro:sensor_hokuyo parent="base_link" xyz="${base_len/2 + 0.025 + 0.0159} 0 ${0.02 - base_height/2}" rpy="3.14 0 0" />
+  <xacro:sensor_hokuyo parent="base_link" xyz="${base_len/2 + 0.017 + 0.024} 0 ${0.02 - base_height/2}" rpy="3.14 0 0" name="front"/>
+  <xacro:sensor_hokuyo parent="base_link" xyz="${-base_len/2 - 0.017 - 0.024} 0 ${0.02 - base_height/2}" rpy="3.14 0 3.14" name="back"/>
 </robot>

Commit message: new URDF working

File: urdf/shark_v1.xacro (robot description, xacro)
@@ -4,7 +4,7 @@
   <xacro:property name="base_width" value="0.335"/>
   <xacro:property name="base_len" value="0.5"/>
-  <xacro:property name="base_height" value="0.3"/>
+  <xacro:property name="base_height" value="0.235"/>
   <xacro:property name="wheel_radius" value="0.1"/>
-  <xacro:property name="base_wheel_gap" value="0.005"/>
+  <xacro:property name="base_wheel_gap" value="0.03"/>
   <xacro:property name="wheel_separation" value="0.36"/>
   <xacro:property name="wheel_joint_offset" value="0.0"/>

Commit message: added imu link

File: urdf/shark_v1.xacro (robot description, xacro)
@@ -106,4 +106,12 @@
     </inertial>
   </xacro:macro>
+  <xacro:macro name="imu" params="parent xyz rpy">
+    <link name="imu_link"/>
+    <joint name="imu_joint" type="fixed">
+      <parent link="${parent}"/>
+      <child link="imu_link"/>
+      <origin xyz="${xyz}" rpy="${rpy}"/>
+    </joint>
+  </xacro:macro>
    <!-- <link name="caster_wheel">
      <visual>
@@ -130,3 +138,4 @@
   <xacro:sensor_hokuyo parent="base_link" xyz="${base_len/2 + 0.017 + 0.024} 0 ${0.02 - base_height/2}" rpy="3.14 0 0" name="front"/>
   <xacro:sensor_hokuyo parent="base_link" xyz="${-base_len/2 - 0.017 - 0.024} 0 ${0.02 - base_height/2}" rpy="3.14 0 3.14" name="back"/>
+  <xacro:imu parent="base_link" xyz="${base_len/2 + 0.0625} 0 ${0.02 - base_height/2}" rpy="0 0 0"/>
 </robot>

Commit message: corredor test, good result

File: urdf/shark_v1.xacro (robot description, xacro)
@@ -7,5 +7,5 @@
   <xacro:property name="wheel_radius" value="0.1"/>
   <xacro:property name="base_wheel_gap" value="0.03"/>
-  <xacro:property name="wheel_separation" value="0.36"/>
+  <xacro:property name="wheel_separation" value="0.4"/>
   <xacro:property name="wheel_joint_offset" value="0.0"/>
   <xacro:property name="caster_height" value="0.07"/>

Commit message: localization with two hokuyos working

File: urdf/shark_v1.xacro (robot description, xacro)
@@ -1,13 +1,13 @@
 <?xml version="1.0"?>
 <robot xmlns:xacro="http://www.ros.org/wiki/xacro" name="shark-v1">
-  <xacro:include filename="$(find doris_sensors_description)/urdf/hokuyo.urdf.xacro" />
-  <xacro:property name="base_width" value="0.531"/>
-  <xacro:property name="base_len" value="0.3785"/>
-  <xacro:property name="base_height" value="0.2895"/>
+  <xacro:include filename="$(find doris_sensors_description)/urdf/hokuyo.urdf.xacro"/>
+  <xacro:property name="base_width" value="0.335"/>
+  <xacro:property name="base_len" value="0.5"/>
+  <xacro:property name="base_height" value="0.235"/>
   <xacro:property name="wheel_radius" value="0.1"/>
-  <xacro:property name="base_wheel_gap" value="-0.09"/>
-  <xacro:property name="wheel_separation" value="0.35"/>
-  <xacro:property name="wheel_joint_offset" value="-0.005"/>
-  <xacro:property name="caster_height" value="0.060575"/>
+  <xacro:property name="base_wheel_gap" value="0.03"/>
+  <xacro:property name="wheel_separation" value="0.36"/>
+  <xacro:property name="wheel_joint_offset" value="0.0"/>
+  <xacro:property name="caster_height" value="0.07"/>
   <!-- <xacro:property name="caster_wheel_radius" value="0.0375"/>
   <xacro:property name="caster_wheel_joint_offset" value="0.12"/> -->
@@ -40,5 +40,5 @@
   </xacro:macro>
   <link name="base_footprint">
-    <!-- <xacro:box_inertia m="8" w="0.001" h="0.001" d="0.001"/> -->
+    <xacro:box_inertia m="8" w="0.001" h="0.001" d="0.001"/>
     <visual>
       <origin xyz="0 0 0" rpy="0 0 0" />
@@ -128,4 +128,5 @@
     <origin xyz="${caster_wheel_joint_offset} 0 -${0.06+caster_wheel_radius}" rpy="0 0 0"/>
   </joint> -->
-  <xacro:sensor_hokuyo parent="base_link" xyz="${base_len/2 + 0.025 + 0.0159} 0 ${0.02 - base_height/2}" rpy="3.14 0 0" />
+  <xacro:sensor_hokuyo parent="base_link" xyz="${base_len/2 + 0.017 + 0.024} 0 ${0.02 - base_height/2}" rpy="3.14 0 0" name="front"/>
+  <xacro:sensor_hokuyo parent="base_link" xyz="${-base_len/2 - 0.017 - 0.024} 0 ${0.02 - base_height/2}" rpy="3.14 0 3.14" name="back"/>
 </robot>

Commit message: added body_scan but need to test

File: urdf/shark_v1.xacro (robot description, xacro)
@@ -106,4 +106,12 @@
     </inertial>
   </xacro:macro>
+  <xacro:macro name="imu" params="parent xyz rpy">
+    <link name="imu_link"/>
+    <joint name="imu_joint" type="fixed">
+      <parent link="${parent}"/>
+      <child link="imu_link"/>
+      <origin xyz="${xyz}" rpy="${rpy}"/>
+    </joint>
+  </xacro:macro>
    <!-- <link name="caster_wheel">
      <visual>
@@ -128,5 +136,7 @@
     <origin xyz="${caster_wheel_joint_offset} 0 -${0.06+caster_wheel_radius}" rpy="0 0 0"/>
   </joint> -->
-  <xacro:sensor_hokuyo parent="base_link" xyz="${base_len/2 + 0.017 + 0.024} 0 ${0.02 - base_height/2}" rpy="3.14 0 0" name="front"/>
+  <xacro:sensor_hokuyo parent="base_link" xyz="${base_len/2 + 0.017 + 0.024} 0 ${base_height/2}" rpy="0 0 0" name="body"/>
+  <xacro:sensor_hokuyo parent="base_link" xyz="${base_len/2 + 0.017 + 0.024} 0 ${0.02 - base_height/2}" rpy="3.14 0 0" name="ground"/>
   <xacro:sensor_hokuyo parent="base_link" xyz="${-base_len/2 - 0.017 - 0.024} 0 ${0.02 - base_height/2}" rpy="3.14 0 3.14" name="back"/>
+  <xacro:imu parent="base_link" xyz="${base_len/2 + 0.0625} 0 ${0.02 - base_height/2}" rpy="0 0 0"/>
 </robot>

Commit message: changed main laser to sick

File: urdf/shark_v1.xacro (robot description, xacro)
@@ -2,4 +2,5 @@
 <robot xmlns:xacro="http://www.ros.org/wiki/xacro" name="shark-v1">
   <xacro:include filename="$(find doris_sensors_description)/urdf/hokuyo.urdf.xacro"/>
+  <xacro:include filename="$(find doris_sensors_description)/urdf/sick_lms1xx.urdf.xacro"/>
   <xacro:property name="base_width" value="0.335"/>
   <xacro:property name="base_len" value="0.5"/>
@@ -136,5 +137,11 @@
     <origin xyz="${caster_wheel_joint_offset} 0 -${0.06+caster_wheel_radius}" rpy="0 0 0"/>
   </joint> -->
-  <xacro:sensor_hokuyo parent="base_link" xyz="${base_len/2 + 0.017 + 0.024} 0 ${base_height/2}" rpy="0 0 0" name="body"/>
+  <!-- <xacro:sensor_hokuyo parent="base_link" xyz="${base_len/2 + 0.017 + 0.024} 0 ${base_height/2}" rpy="0 0 0" name="body"/> -->
+  <xacro:sick_lms1xx/>
+  <joint name="laser_joint" type="fixed">
+    <origin xyz="${base_len/2 + 0.017 + 0.05} 0 ${0.02 + base_height/2}" rpy="0 0 0" />
+    <parent link="base_link" />
+    <child link="sick_link" />
+  </joint>
   <xacro:sensor_hokuyo parent="base_link" xyz="${base_len/2 + 0.017 + 0.024} 0 ${0.02 - base_height/2}" rpy="3.14 0 0" name="ground"/>
   <xacro:sensor_hokuyo parent="base_link" xyz="${-base_len/2 - 0.017 - 0.024} 0 ${0.02 - base_height/2}" rpy="3.14 0 3.14" name="back"/>
