Commit message: adjusted to tests in the robot

File: urdf/shark_v1.xacro (robot description, xacro)
@@ -1,64 +1,75 @@
 <?xml version="1.0"?>
 <robot xmlns:xacro="http://www.ros.org/wiki/xacro" name="shark-v1">
-  <xacro:include filename="$(find doris_sensors_description)/urdf/hokuyo.urdf.xacro"/>
-  <xacro:include filename="$(find doris_sensors_description)/urdf/sick_lms1xx.urdf.xacro"/>
-  <xacro:property name="base_width" value="0.335"/>
-  <xacro:property name="base_len" value="0.5"/>
-  <xacro:property name="base_height" value="0.235"/>
-  <xacro:property name="wheel_radius" value="0.1"/>
-  <xacro:property name="base_wheel_gap" value="0.03"/>
-  <xacro:property name="wheel_separation" value="0.36"/>
-  <xacro:property name="wheel_joint_offset" value="0.0"/>
-  <xacro:property name="caster_height" value="0.07"/>
+  <xacro:include filename="$(find doris_sensors_description)/urdf/hokuyo.urdf.xacro" />
+  <xacro:include filename="$(find doris_sensors_description)/urdf/sick_lms1xx.urdf.xacro" />
+  <xacro:include filename="$(find doris_sensors_description)/urdf/realsense_camera.urdf.xacro" />
+  <xacro:include filename="$(find hector_sensors_description)/urdf/realsense_d435_camera.urdf.xacro" />
+  <xacro:include filename="$(find doris_head_description)/urdf/doris_head.urdf" />
+  <xacro:property name="base_width" value="0.335" />
+  <xacro:property name="base_len" value="0.5" />
+  <xacro:property name="base_height" value="0.235" />
+  <xacro:property name="wheel_radius" value="0.1" />
+  <xacro:property name="base_wheel_gap" value="0.03" />
+  <xacro:property name="wheel_separation" value="0.36" />
+  <xacro:property name="wheel_joint_offset" value="0.0" />
+  <xacro:property name="caster_height" value="0.07" />
+  <xacro:property name="dorso_width" value="0.337" />
+  <xacro:property name="dorso_len" value="0.28" />
+  <xacro:property name="dorso_height" value="0.8" />
+  <xacro:property name="arm_support_width" value="0.34" />
+  <xacro:property name="arm_support_len" value="0.33" />
+  <xacro:property name="arm_support_height" value="0.04" />
+  <xacro:property name="arm_z_position" value="0.51" />
   <!-- <xacro:property name="caster_wheel_radius" value="0.0375"/>
   <xacro:property name="caster_wheel_joint_offset" value="0.12"/> -->
-  <xacro:include filename="$(find shark-mb-ros)/urdf/shark_v1_gazebo_plugins.xacro"/>
+  <xacro:include filename="$(find shark-mb-ros)/urdf/shark_v1_gazebo_plugins.xacro" />
   <material name="blue">
-    <color rgba="0 0 0.8 1"/>
+    <color rgba="0 0 0.8 1" />
   </material>
   <material name="black">
-    <color rgba="0 0 0 1"/>
+    <color rgba="0 0 0 1" />
   </material>
   <material name="darkgray">
-    <color rgba="0.2 0.2 0.2 1"/>
+    <color rgba="0.2 0.2 0.2 1" />
   </material>
   <material name="lightgray">
-    <color rgba="0.8 0.8 0.8 1"/>
+    <color rgba="0.8 0.8 0.8 1" />
   </material>
   <material name="white">
-    <color rgba="1 1 1 1"/>
+    <color rgba="1 1 1 1" />
   </material>
   <material name="red">
-    <color rgba="0.8 0.0 0.0 1.0"/>
+    <color rgba="0.8 0.0 0.0 1.0" />
   </material>
   <!-- Import Rviz colors -->
-<!--  <xacro:include filename="$(find ros_robotics)/urdf/materials.xacro" /> -->
+  <!--  <xacro:include filename="$(find ros_robotics)/urdf/materials.xacro" /> -->
   <xacro:macro name="box_inertia" params="m w h d">
     <inertial>
-      <mass value="${m}"/>
-      <inertia ixx="${m / 12.0 * (d*d + h*h)}" ixy="0.0" ixz="0.0" iyy="${m / 12.0 * (w*w + h*h)}" iyz="0.0" izz="${m / 12.0 * (w*w + d*d)}"/>
+      <mass value="${m}" />
+      <inertia ixx="${m / 12.0 * (d*d + h*h)}" ixy="0.0" ixz="0.0" iyy="${m / 12.0 * (w*w + h*h)}"
+        iyz="0.0" izz="${m / 12.0 * (w*w + d*d)}" />
     </inertial>
   </xacro:macro>
   <link name="base_footprint">
-    <xacro:box_inertia m="8" w="0.001" h="0.001" d="0.001"/>
+    <xacro:box_inertia m="8" w="0.001" h="0.001" d="0.001" />
     <visual>
       <origin xyz="0 0 0" rpy="0 0 0" />
-      <material name="white"/>
-        <geometry>
-            <box size="0.001 0.001 0.001" />
-        </geometry>
+      <material name="white" />
+      <geometry>
+        <box size="0.001 0.001 0.001" />
+      </geometry>
     </visual>
   </link>
   <link name="base_link">
-    <xacro:box_inertia m="1" w="${base_len}" h="${base_width}" d="0.01"/>
+    <xacro:box_inertia m="1" w="${base_len}" h="${base_width}" d="0.01" />
     <visual>
-      <material name="lightgray"/>
+      <material name="lightgray" />
       <geometry>
-        <box size="${base_len} ${base_width} ${base_height}"/>
+        <box size="${base_len} ${base_width} ${base_height}" />
       </geometry>
     </visual>
     <collision>
       <geometry>
-        <box size="${base_len} ${base_width} ${base_height}"/>
+        <box size="${base_len} ${base_width} ${base_height}" />
       </geometry>
     </collision>
@@ -66,11 +77,12 @@
   <joint name="base_link_joint" type="fixed">
     <origin xyz="0 0 ${base_height/2 + caster_height}" rpy="0 0 0" />
-    <parent link="base_footprint"/>
+    <parent link="base_footprint" />
     <child link="base_link" />
   </joint>
   <xacro:macro name="cylinder_inertia" params="m r h">
     <inertial>
-      <mass value="${m}"/>
-      <inertia ixx="${m*(3*r*r+h*h)/12}" ixy = "0" ixz = "0" iyy="${m*(3*r*r+h*h)/12}" iyz = "0" izz="${m*r*r/2}"/>
+      <mass value="${m}" />
+      <inertia ixx="${m*(3*r*r+h*h)/12}" ixy="0" ixz="0" iyy="${m*(3*r*r+h*h)/12}" iyz="0"
+        izz="${m*r*r/2}" />
     </inertial>
   </xacro:macro>
@@ -78,65 +90,90 @@
     <link name="${prefix}_wheel">
       <visual>
-	<material name="darkgray"/>
-        <origin xyz="0 0 0" rpy="${pi/2} 0 0"/>
+        <material name="darkgray" />
+        <origin xyz="0 0 0" rpy="${pi/2} 0 0" />
         <geometry>
-          <cylinder radius="${wheel_radius}" length="0.05"/>
+          <cylinder radius="${wheel_radius}" length="0.05" />
         </geometry>
       </visual>
       <collision>
-        <origin xyz="0 0 0" rpy="${pi/2} 0 0"/>
+        <origin xyz="0 0 0" rpy="${pi/2} 0 0" />
         <geometry>
-          <cylinder radius="${wheel_radius}" length="0.05"/>
+          <cylinder radius="${wheel_radius}" length="0.05" />
         </geometry>
       </collision>
-      <xacro:cylinder_inertia m="10" r="${wheel_radius}" h="0.05"/>
+      <xacro:cylinder_inertia m="10" r="${wheel_radius}" h="0.05" />
     </link>
     <joint name="${prefix}_wheel" type="continuous">
       <axis xyz="0 1 0" rpy="0 0 0" />
-      <parent link="base_link"/>
-      <child link="${prefix}_wheel"/>
-      <origin xyz="${wheel_joint_offset} ${((base_width/2)+base_wheel_gap)*reflect} ${(wheel_radius - caster_height) - base_height/2}" rpy="0 0 0"/>
+      <parent link="base_link" />
+      <child link="${prefix}_wheel" />
+      <origin
+        xyz="${wheel_joint_offset} ${((base_width/2)+base_wheel_gap)*reflect} ${(wheel_radius - caster_height) - base_height/2}"
+        rpy="0 0 0" />
     </joint>
   </xacro:macro>
-  <xacro:wheel prefix="left" reflect="1"/>
-  <xacro:wheel prefix="right" reflect="-1"/>
+  <xacro:wheel prefix="left" reflect="1" />
+  <xacro:wheel prefix="right" reflect="-1" />
   <xacro:macro name="sphere_inertia" params="m r">
     <inertial>
-      <mass value="${m}"/>
-      <inertia ixx="${2.0*m*(r*r)/5.0}" ixy="0.0" ixz="0.0" iyy="${2.0*m*(r*r)/5.0}" iyz="0.0" izz="${2.0*m*(r*r)/5.0}"/>
+      <mass value="${m}" />
+      <inertia ixx="${2.0*m*(r*r)/5.0}" ixy="0.0" ixz="0.0" iyy="${2.0*m*(r*r)/5.0}" iyz="0.0"
+        izz="${2.0*m*(r*r)/5.0}" />
     </inertial>
   </xacro:macro>
   <xacro:macro name="imu" params="parent xyz rpy">
-    <link name="imu_link"/>
+    <link name="imu_link" />
     <joint name="imu_joint" type="fixed">
-      <parent link="${parent}"/>
-      <child link="imu_link"/>
-      <origin xyz="${xyz}" rpy="${rpy}"/>
+      <parent link="${parent}" />
+      <child link="imu_link" />
+      <origin xyz="${xyz}" rpy="${rpy}" />
     </joint>
   </xacro:macro>
-   <!-- <link name="caster_wheel">
-     <visual>
-       <material name="darkgray"/>
-      <origin xyz="0 0 0" rpy="0 0 0"/>
-      <geometry>
-        <sphere radius="${caster_wheel_radius}"/>
-      </geometry>
-    </visual>
-    <collision>
-      <origin xyz="0 0 0" rpy="0 0 0"/>
-      <geometry>
-        <sphere radius="${caster_wheel_radius}"/>
-      </geometry>
-    </collision>
-    <xacro:sphere_inertia m="5" r="${caster_wheel_radius}"/>
-  </link>
-  <joint name="caster_wheel_joint" type="continuous">
-    <axis xyz="0 1 0" rpy="0 0 0" />
-    <parent link="base_link"/>
-    <child link="caster_wheel"/>
-    <origin xyz="${caster_wheel_joint_offset} 0 -${0.06+caster_wheel_radius}" rpy="0 0 0"/>
-  </joint> -->
-  <!-- <xacro:sensor_hokuyo parent="base_link" xyz="${base_len/2 + 0.017 + 0.024} 0 ${base_height/2}" rpy="0 0 0" name="body"/> -->
-  <xacro:sick_lms1xx/>
+  <xacro:sick_lms1xx />
+  <xacro:macro name="dorso" params="parent depth width height xyz rpy">
+    <link name="dorso_link">
+      <xacro:box_inertia m="1" w="${width}" h="${height}" d="0.01" />
+      <visual>
+        <origin xyz="0.0 0.0 ${height/2}"/>
+        <material name="lightgray" />
+        <geometry>
+          <box size="${depth} ${width} ${height}" />
+          </geometry>
+          </visual>
+          <collision>
+            <origin xyz="0.0 0.0 ${height/2}"/>
+            <geometry>
+              <box size="${depth} ${width} ${height}" />
+              </geometry>
+      </collision>
+    </link>
+    <joint name="dorso_joint" type="fixed">
+        <parent link="${parent}"/>
+        <child link="dorso_link"/>
+        <origin xyz="${xyz}" rpy="${rpy}"/>
+    </joint>
+  </xacro:macro>
+    <!--32,5-->
+  <xacro:macro name="arm_support" params="parent width height depth xyz rpy">
+    <link name="arm_support_link">
+      <xacro:box_inertia m="1" w="${width}" h="${height}" d="0.01" />
+      <visual>
+        <material name="lightgray" />
+        <geometry>
+          <box size="${depth} ${width} ${height}" />
+        </geometry>
+      </visual>
+      <collision>
+        <geometry>
+          <box size="${depth} ${width} ${height}" />
+        </geometry>
+      </collision>
+    </link>
+    <joint name="arm_support_joint" type="fixed">
+        <parent link="${parent}"/>
+        <child link="arm_support_link"/>
+        <origin xyz="${xyz}" rpy="${rpy}"/>
+    </joint>
+  </xacro:macro>
   <joint name="laser_joint" type="fixed">
     <origin xyz="${base_len/2 + 0.017 + 0.05} 0 ${0.02 + base_height/2}" rpy="0 0 0" />
@@ -144,6 +181,16 @@
     <child link="sick_link" />
   </joint>
+  <joint name="dorso_head" type="fixed">
+    <parent link="dorso_link" />
+    <child link="head_root" />
+    <origin xyz="0 0 ${dorso_height + 0.04}" rpy="0 0 0" />
+  </joint>
+  <xacro:realsense_camera name="camera" parent="dorso_link">
+    <origin xyz="${dorso_len/2 - 0.063} 0 ${dorso_height}" rpy="0 0 0" />
+  </xacro:realsense_camera>
+  <xacro:dorso parent="base_link" depth="${dorso_len}" width="${dorso_width}" height="${dorso_height}" xyz="${-base_len/2 + (dorso_len/2)} 0 ${base_height/2}" rpy="0 0 0"/>
+  <xacro:arm_support parent="dorso_link" width="${arm_support_width}" height="${arm_support_height}" depth="${arm_support_len}" xyz="${dorso_len/2 + arm_support_len/2} 0 ${arm_z_position}" rpy="0 0 0"/>
   <xacro:sensor_hokuyo parent="base_link" xyz="${base_len/2 + 0.017 + 0.024} 0 ${0.02 - base_height/2}" rpy="3.14 0 0" name="ground"/>
   <xacro:sensor_hokuyo parent="base_link" xyz="${-base_len/2 - 0.017 - 0.024} 0 ${0.02 - base_height/2}" rpy="3.14 0 3.14" name="back"/>
-  <xacro:imu parent="base_link" xyz="${base_len/2 + 0.0625} 0 ${0.02 - base_height/2}" rpy="0 0 0"/>
+  <xacro:imu parent="base_link" xyz="${base_len/2 + 0.0625} 0 ${0.02 - base_height/2}" rpy="0 0 0" />
 </robot>

Commit message: :construction: checkpoint: need to move arm to correct place

File: urdf/shark_v1.xacro (robot description, xacro)
@@ -6,4 +6,7 @@
   <xacro:include filename="$(find hector_sensors_description)/urdf/realsense_d435_camera.urdf.xacro" />
   <xacro:include filename="$(find doris_head_description)/urdf/doris_head.urdf" />
+  <xacro:macro name="wx200" params="parent 10 10 10 rpy name">
+    <xacro:include filename="$(find interbotix_xsarm_descriptions)/urdf/mobile_wx200.urdf.xacro" />
+  </xacro:macro>
   <xacro:property name="base_width" value="0.335" />
   <xacro:property name="base_len" value="0.5" />
@@ -194,3 +197,4 @@
   <xacro:sensor_hokuyo parent="base_link" xyz="${-base_len/2 - 0.017 - 0.024} 0 ${0.02 - base_height/2}" rpy="3.14 0 3.14" name="back"/>
   <xacro:imu parent="base_link" xyz="${base_len/2 + 0.0625} 0 ${0.02 - base_height/2}" rpy="0 0 0" />
+  <xacro:wx200 parent="dorso_link" xyz="10 10 10" rpy="0 0 0" name="wx200"/>
 </robot>

Commit message: fixed boris arm position

File: urdf/shark_v1.xacro (robot description, xacro)
@@ -6,7 +6,5 @@
   <xacro:include filename="$(find hector_sensors_description)/urdf/realsense_d435_camera.urdf.xacro" />
   <xacro:include filename="$(find doris_head_description)/urdf/doris_head.urdf" />
-  <xacro:macro name="wx200" params="parent 10 10 10 rpy name">
-    <xacro:include filename="$(find interbotix_xsarm_descriptions)/urdf/mobile_wx200.urdf.xacro" />
-  </xacro:macro>
+  <xacro:include filename="$(find interbotix_xsarm_descriptions)/urdf/boris_arm.xacro" />
   <xacro:property name="base_width" value="0.335" />
   <xacro:property name="base_len" value="0.5" />
@@ -155,5 +153,5 @@
         <child link="dorso_link"/>
         <origin xyz="${xyz}" rpy="${rpy}"/>
-    </joint>
+    </joint>0
   </xacro:macro>
     <!--32,5-->
@@ -197,4 +195,4 @@
   <xacro:sensor_hokuyo parent="base_link" xyz="${-base_len/2 - 0.017 - 0.024} 0 ${0.02 - base_height/2}" rpy="3.14 0 3.14" name="back"/>
   <xacro:imu parent="base_link" xyz="${base_len/2 + 0.0625} 0 ${0.02 - base_height/2}" rpy="0 0 0" />
-  <xacro:wx200 parent="dorso_link" xyz="10 10 10" rpy="0 0 0" name="wx200"/>
+  <xacro:boris_arm parent="arm_support_link" xyz="0.1 0 ${arm_support_height/2}" rpy="0 0 0"/>
 </robot>

Commit message: added arm support height as argument

File: urdf/shark_v1.xacro (robot description, xacro)
@@ -7,4 +7,5 @@
   <xacro:include filename="$(find doris_head_description)/urdf/doris_head.urdf" />
   <xacro:include filename="$(find interbotix_xsarm_descriptions)/urdf/wx200.urdf.xacro" />
+  <xacro:arg name="arm_z_position" default="0.51"/>
   <xacro:property name="base_width" value="0.335" />
   <xacro:property name="base_len" value="0.5" />
@@ -21,5 +22,5 @@
   <xacro:property name="arm_support_len" value="0.33" />
   <xacro:property name="arm_support_height" value="0.04" />
-  <xacro:property name="arm_z_position" value="0.51" />
+  <xacro:property name="arm_z_position" value="$(arg arm_z_position)" />
   <!-- <xacro:property name="caster_wheel_radius" value="0.0375"/>
   <xacro:property name="caster_wheel_joint_offset" value="0.12"/> -->

Commit message: changed wheels distance

File: urdf/shark_v1.xacro (robot description, xacro)
@@ -11,5 +11,5 @@
   <xacro:property name="base_height" value="0.235" />
   <xacro:property name="wheel_radius" value="0.1" />
-  <xacro:property name="base_wheel_gap" value="0.03" />
+  <xacro:property name="base_wheel_gap" value="0.035" />
   <xacro:property name="wheel_separation" value="0.36" />
   <xacro:property name="wheel_joint_offset" value="0.0" />
@@ -194,5 +194,5 @@
   <xacro:sensor_hokuyo parent="base_link" xyz="${base_len/2 + 0.017 + 0.024} 0 ${0.02 - base_height/2}" rpy="3.14 0 0" name="ground"/>
   <xacro:sensor_hokuyo parent="base_link" xyz="${-base_len/2 - 0.017 - 0.024} 0 ${0.02 - base_height/2}" rpy="3.14 0 3.14" name="back"/>
-  <xacro:imu parent="base_link" xyz="-0.01 0 ${0.02 - base_height/2}" rpy="0 0 0" />
+  <xacro:imu parent="base_link" xyz="-0.01 0 ${0.02 - base_height/2}" rpy="-0.0041582 -0.0710581 0" />
   <xacro:boris_arm parent="arm_support_link" xyz="0.1 0 ${arm_support_height/2}" rpy="0 0 0"/>
 </robot>

Commit message: changed wheels params

File: urdf/shark_v1.xacro (robot description, xacro)
@@ -11,6 +11,6 @@
   <xacro:property name="base_len" value="0.5" />
   <xacro:property name="base_height" value="0.235" />
-  <xacro:property name="wheel_radius" value="0.1" />
-  <xacro:property name="base_wheel_gap" value="0.035" />
+  <xacro:property name="wheel_radius" value="0.105" />
+  <xacro:property name="base_wheel_gap" value="0.075" />
   <xacro:property name="wheel_separation" value="0.36" />
   <xacro:property name="wheel_joint_offset" value="0.0" />

Commit message: changed footprints

File: urdf/shark_v1.xacro (robot description, xacro)
@@ -95,5 +95,5 @@
         <origin xyz="0 0 0" rpy="${pi/2} 0 0" />
         <geometry>
-          <cylinder radius="${wheel_radius}" length="0.05" />
+          <cylinder radius="${wheel_radius}" length="0.1" />
         </geometry>
       </visual>

Commit message: changed realsense x and z position

File: urdf/shark_v1.xacro (robot description, xacro)
@@ -189,5 +189,5 @@
   </joint>
   <xacro:realsense_camera name="camera" parent="dorso_link">
-    <origin xyz="${dorso_len/2 - 0.063} 0 ${dorso_height}" rpy="0 0 0" />
+    <origin xyz="${dorso_len/2 + 0.05} 0 ${dorso_height + 0.053}" rpy="0 0 0" />
   </xacro:realsense_camera>
   <xacro:dorso parent="base_link" depth="${dorso_len}" width="${dorso_width}" height="${dorso_height}" xyz="${-base_len/2 + (dorso_len/2)} 0 ${base_height/2}" rpy="0 0 0"/>

Commit message: changed hoverboard wheels

File: urdf/shark_v1.xacro (robot description, xacro)
@@ -11,7 +11,7 @@
   <xacro:property name="base_len" value="0.5" />
   <xacro:property name="base_height" value="0.235" />
-  <xacro:property name="wheel_radius" value="0.105" />
-  <xacro:property name="base_wheel_gap" value="0.075" />
-  <xacro:property name="wheel_separation" value="0.36" />
+  <xacro:property name="wheel_radius" value="0.0825" />
+  <xacro:property name="base_wheel_gap" value="0.07" />
+  <xacro:property name="wheel_separation" value="0.39" />
   <xacro:property name="wheel_joint_offset" value="0.0" />
   <xacro:property name="caster_height" value="0.07" />

Commit message: adjusted wheel width

File: urdf/shark_v1.xacro (robot description, xacro)
@@ -12,5 +12,6 @@
   <xacro:property name="base_height" value="0.235" />
   <xacro:property name="wheel_radius" value="0.0825" />
-  <xacro:property name="base_wheel_gap" value="0.07" />
+  <xacro:property name="base_wheel_gap" value="0.05" />
+  <xacro:property name="wheel_width" value="0.06" />
   <xacro:property name="wheel_separation" value="0.39" />
   <xacro:property name="wheel_joint_offset" value="0.0" />
@@ -95,5 +96,5 @@
         <origin xyz="0 0 0" rpy="${pi/2} 0 0" />
         <geometry>
-          <cylinder radius="${wheel_radius}" length="0.1" />
+          <cylinder radius="${wheel_radius}" length="${wheel_width}" />
         </geometry>
       </visual>

Commit message: :zap: URDF updated

File: urdf/shark_v1.xacro (robot description, xacro)
@@ -7,8 +7,7 @@
   <xacro:include filename="$(find doris_head_description)/urdf/doris_head.urdf" />
   <xacro:include filename="$(find interbotix_xsarm_descriptions)/urdf/wx200.urdf.xacro" />
-  <xacro:arg name="arm_z_position" default="0.48"/>
-  <xacro:property name="base_width" value="0.335" />
+  <xacro:property name="base_width" value="0.336" />
   <xacro:property name="base_len" value="0.5" />
-  <xacro:property name="base_height" value="0.235" />
+  <xacro:property name="base_height" value="0.231" />
   <xacro:property name="wheel_radius" value="0.0825" />
   <xacro:property name="base_wheel_gap" value="0.05" />
@@ -17,11 +16,12 @@
   <xacro:property name="wheel_joint_offset" value="0.0" />
   <xacro:property name="caster_height" value="0.07" />
-  <xacro:property name="dorso_width" value="0.337" />
-  <xacro:property name="dorso_len" value="0.28" />
-  <xacro:property name="dorso_height" value="0.8" />
-  <xacro:property name="arm_support_width" value="0.34" />
-  <xacro:property name="arm_support_len" value="0.33" />
-  <xacro:property name="arm_support_height" value="0.04" />
+  <xacro:property name="dorso_width" value="0.338" />
+  <xacro:property name="dorso_len" value="0.282" />
+  <xacro:property name="dorso_height" value="0.765" />
+  <xacro:property name="arm_support_width" value="0.336" />
+  <xacro:property name="arm_support_len" value="0.325" />
+  <xacro:property name="arm_support_height" value="0.047" />
   <xacro:property name="arm_z_position" value="$(arg arm_z_position)" />
+  <xacro:arg name="arm_z_position" default="0.34"/>
   <!-- <xacro:property name="caster_wheel_radius" value="0.0375"/>
   <xacro:property name="caster_wheel_joint_offset" value="0.12"/> -->

Commit message: added webcam to arm

File: urdf/shark_v1.xacro (robot description, xacro)
@@ -179,4 +179,43 @@
     </joint>
   </xacro:macro>
+  <xacro:macro name="rgb_cam" params="parent name xyz rpy">
+    <link name="${name}_link">
+      <visual>
+        <material name="lightgray"/>
+        <geometry>
+          <box size="0.013 0.0627 0.02597"/>
+        </geometry>
+      </visual>
+      <collision>
+        <geometry>
+          <box size="0.013 0.0627 0.02597"/>
+        </geometry>
+      </collision>
+    </link>
+    <link name="${name}_lens_link">
+      <visual>
+        <material name="black"/>
+        <origin rpy="0.0 1.5707963267948966 0.0"/>
+        <geometry>
+          <cylinder radius="0.00725" length="0.015"/>
+        </geometry>
+      </visual>
+      <collision>
+        <geometry>
+          <cylinder radius="0.00725" length="0.015"/>
+        </geometry>
+      </collision>
+    </link>
+    <joint name="${name}_joint" type="fixed">
+      <parent link="${parent}"/>
+      <child link="${name}_link"/>
+      <origin xyz="${xyz}" rpy="${rpy}"/>
+    </joint>
+    <joint name="${name}_lens_joint" type="fixed">
+      <parent link="${name}_link"/>
+      <child link="${name}_lens_link"/>
+      <origin xyz="0.0 0.015375 0.0"/>
+    </joint>
+  </xacro:macro>
   <joint name="laser_joint" type="fixed">
     <origin xyz="${base_len/2 + 0.017 + 0.05} 0 ${0.02 + base_height/2}" rpy="0 0 0" />
@@ -198,3 +237,4 @@
   <xacro:imu parent="base_link" xyz="-0.01 0 ${0.02 - base_height/2}" rpy="-0.014161 -0.0203861 0" />
   <xacro:boris_arm parent="arm_support_link" xyz="0.1 0 ${arm_support_height/2}" rpy="0 0 0"/>
+  <xacro:rgb_cam parent="wx200/gripper_bar_link" name="webcam" xyz="-0.078 0.0 0.05" rpy="0 0 0"/>
 </robot>
