Commit message: changed lens position

File: urdf/shark_v1.xacro (robot description, xacro)
@@ -196,12 +196,12 @@
       <visual>
         <material name="black"/>
-        <origin rpy="0.0 1.5707963267948966 0.0"/>
-        <geometry>
-          <cylinder radius="0.00725" length="0.015"/>
-        </geometry>
-      </visual>
-      <collision>
-        <geometry>
-          <cylinder radius="0.00725" length="0.015"/>
+        <origin xyz="0.001 0 0" rpy="0.0 1.5707963267948966 0.0"/>
+        <geometry>
+          <cylinder radius="0.00725" length="0.013"/>
+        </geometry>
+      </visual>
+      <collision>
+        <geometry>
+          <cylinder radius="0.00725" length="0.013"/>
         </geometry>
       </collision>
@@ -215,5 +215,5 @@
       <parent link="${name}_link"/>
       <child link="${name}_lens_link"/>
-      <origin xyz="0.0 0.015375 0.0"/>
+      <origin xyz="0.0 -0.015375 0.0"/>
     </joint>
   </xacro:macro>
